Commit message: updated lower/upper servo range limits

File: src/hexapod_model_description/urdf/hexapod_model.xacro (robot description, xacro)
@@ -426,5 +426,5 @@
     <child link="leg1_coxa_1"/>
     <axis xyz="-0.0 0.0 1.0"/>
-    <limit lower="0.0" upper="3.14159" effort="100" velocity="1.0" />
+    <limit lower="-1.57" upper="1.57" effort="100" velocity="1.0" />
   </joint>
   <joint name="leg1_femur_joint" type="revolute">
@@ -433,5 +433,5 @@
     <child link="leg1_femur_1"/>
     <axis xyz="-0.573576 -0.819152 -0.0"/>
-    <limit lower="0.0" upper="3.14159" effort="100" velocity="1.0" />
+    <limit lower="-1.57" upper="1.57" effort="100" velocity="1.0" />
   </joint>
   <joint name="leg1_tibia_joint" type="revolute">
@@ -440,5 +440,5 @@
     <child link="leg1_tibia_1"/>
     <axis xyz="-0.573576 -0.819152 -0.0"/>
-    <limit lower="0.0" upper="3.14159" effort="100" velocity="1.0" />
+    <limit lower="-1.57" upper="1.57" effort="100" velocity="1.0" />
   </joint>
   <joint name="leg2_coxa_joint" type="revolute">
@@ -447,5 +447,5 @@
     <child link="leg2_coxa_1"/>
     <axis xyz="-0.0 0.0 1.0"/>
-    <limit lower="0.0" upper="3.14159" effort="100" velocity="1.0" />
+    <limit lower="-1.57" upper="1.57" effort="100" velocity="1.0" />
   </joint>
   <joint name="leg2_femur_joint" type="revolute">
@@ -454,5 +454,5 @@
     <child link="leg2_femur_1"/>
     <axis xyz="-1.0 0.0 -0.0"/>
-    <limit lower="0.0" upper="3.14159" effort="100" velocity="1.0" />
+    <limit lower="-1.57" upper="1.57" effort="100" velocity="1.0" />
   </joint>
   <joint name="leg2_tibia_joint" type="revolute">
@@ -461,5 +461,5 @@
     <child link="leg2_tibia_1"/>
     <axis xyz="-1.0 0.0 -0.0"/>
-    <limit lower="0.0" upper="3.14159" effort="100" velocity="1.0" />
+    <limit lower="-1.57" upper="1.57" effort="100" velocity="1.0" />
   </joint>
   <joint name="leg3_coxa_joint" type="revolute">
@@ -468,5 +468,5 @@
     <child link="leg3_coxa_1"/>
     <axis xyz="-0.0 0.0 1.0"/>
-    <limit lower="0.0" upper="3.14159" effort="100" velocity="1.0" />
+    <limit lower="-1.57" upper="1.57" effort="100" velocity="1.0" />
   </joint>
   <joint name="leg3_femur_joint" type="revolute">
@@ -475,5 +475,5 @@
     <child link="leg3_femur_1"/>
     <axis xyz="-0.642788 0.766044 -0.0"/>
-    <limit lower="0.0" upper="3.14159" effort="100" velocity="1.0" />
+    <limit lower="-1.57" upper="1.57" effort="100" velocity="1.0" />
   </joint>
   <joint name="leg3_tibia_joint" type="revolute">
@@ -482,5 +482,5 @@
     <child link="leg3_tibia_1"/>
     <axis xyz="0.642788 -0.766044 0.0"/>
-    <limit lower="0.0" upper="3.14159" effort="100" velocity="1.0" />
+    <limit lower="-1.57" upper="1.57" effort="100" velocity="1.0" />
   </joint>
   <joint name="leg4_coxa_joint" type="revolute">
@@ -489,5 +489,5 @@
     <child link="leg4_coxa_1"/>
     <axis xyz="-0.0 0.0 1.0"/>
-    <limit lower="0.0" upper="3.14159" effort="100" velocity="1.0" />
+    <limit lower="-1.57" upper="1.57" effort="100" velocity="1.0" />
   </joint>
   <joint name="leg4_femur_joint" type="revolute">
@@ -496,5 +496,5 @@
     <child link="leg4_femur_1"/>
     <axis xyz="-0.642788 -0.766044 -0.0"/>
-    <limit lower="0.0" upper="3.14159" effort="100" velocity="1.0" />
+    <limit lower="-1.57" upper="1.57" effort="100" velocity="1.0" />
   </joint>
   <joint name="leg4_tibia_joint" type="revolute">
@@ -503,5 +503,5 @@
     <child link="leg4_tibia_1"/>
     <axis xyz="0.642788 0.766044 0.0"/>
-    <limit lower="0.0" upper="3.14159" effort="100" velocity="1.0" />
+    <limit lower="-1.57" upper="1.57" effort="100" velocity="1.0" />
   </joint>
   <joint name="leg5_coxa_joint" type="revolute">
@@ -510,5 +510,5 @@
     <child link="leg5_coxa_1"/>
     <axis xyz="0.0 -0.0 -1.0"/>
-    <limit lower="0.0" upper="3.14159" effort="100" velocity="1.0" />
+    <limit lower="-1.57" upper="1.57" effort="100" velocity="1.0" />
   </joint>
   <joint name="leg5_femur_joint" type="revolute">
@@ -517,5 +517,5 @@
     <child link="leg5_femur_1"/>
     <axis xyz="-1.0 0.0 -0.0"/>
-    <limit lower="0.0" upper="3.14159" effort="100" velocity="1.0" />
+    <limit lower="-1.57" upper="1.57" effort="100" velocity="1.0" />
   </joint>
   <joint name="leg5_tibia_joint" type="revolute">
@@ -524,5 +524,5 @@
     <child link="leg5_tibia_1"/>
     <axis xyz="1.0 -0.0 0.0"/>
-    <limit lower="0.0" upper="3.14159" effort="100" velocity="1.0" />
+    <limit lower="-1.57" upper="1.57" effort="100" velocity="1.0" />
   </joint>
   <joint name="leg6_coxa_joint" type="revolute">
@@ -531,5 +531,5 @@
     <child link="leg6_coxa_1"/>
     <axis xyz="-0.0 0.0 1.0"/>
-    <limit lower="0.0" upper="3.14159" effort="100" velocity="1.0" />
+    <limit lower="-1.57" upper="1.57" effort="100" velocity="1.0" />
   </joint>
   <joint name="leg6_femur_joint" type="revolute">
@@ -538,5 +538,5 @@
     <child link="leg6_femur_1"/>
     <axis xyz="-0.573576 0.819152 -0.0"/>
-    <limit lower="0.0" upper="3.14159" effort="100" velocity="1.0" />
+    <limit lower="-1.57" upper="1.57" effort="100" velocity="1.0" />
   </joint>
   <joint name="leg6_tibia_joint" type="revolute">
@@ -545,5 +545,5 @@
     <child link="leg6_tibia_1"/>
     <axis xyz="0.573576 -0.819152 0.0"/>
-    <limit lower="0.0" upper="3.14159" effort="100" velocity="1.0" />
+    <limit lower="-1.57" upper="1.57" effort="100" velocity="1.0" />
   </joint>
   <joint name="camera_pan_joint" type="revolute">
@@ -552,5 +552,5 @@
     <child link="neck_1"/>
     <axis xyz="0.0 0.0 1.0"/>
-    <limit lower="0.0" upper="3.14159" effort="100" velocity="1.0" />
+    <limit lower="-1.57" upper="1.57" effort="100" velocity="1.0" />
   </joint>
   <joint name="camera_tilt_joint" type="revolute">
@@ -559,5 +559,5 @@
     <child link="face_1"/>
     <axis xyz="-0.0 -1.0 -0.0"/>
-    <limit lower="0.0" upper="3.14159" effort="100" velocity="1.0" />
+    <limit lower="-1.57" upper="1.57" effort="100" velocity="1.0" />
   </joint>
   <ros2_control name="GazeboSimSystem" type="system">
